File: OstronElectronicsStack/OstronElectronicsStack.kicad_sch (KiCad schematic)
At the start: 26 parts

Commit message: rasp
Parts:
- BT1: value (none) -> BS-7-BLUE; footprint (none) -> BS-7-BLUE:BAT_BS-7-BLUE
- BT2: value (none) -> BK-18650-PC6; footprint (none) -> BK-18650-PC6:BAT_BK-18650-PC6
- C1: value (none) -> 1000u; footprint (none) -> Capacitor_THT:CP_Radial_D10.0mm_P5.00mm
- C2: value (none) -> 100u; footprint (none) -> Capacitor_THT:CP_Radial_D6.3mm_P2.50mm
- D1: value (none) -> D; footprint (none) -> Diode_THT:D_5W_P12.70mm_Horizontal
- J1: value (none) -> GSMSERIAL; footprint (none) -> Connector_PinHeader_2.54mm:PinHeader_1x03_P2.54mm_Vertical
- J10: value (none) -> PROG; footprint (none) -> Connector_PinSocket_2.54mm:PinSocket_1x04_P2.54mm_Vertical
- J11: value (none) -> SOLAR; footprint (none) -> TerminalBlock_Phoenix:TerminalBlock_Phoenix_MKDS-1,5-2-5.08_1x02_P5.08mm_Horizontal
- J12: value (none) -> RELAYgsm; footprint (none) -> TerminalBlock_Phoenix:TerminalBlock_Phoenix_MKDS-1,5-3-5.08_1x03_P5.08mm_Horizontal
- J13: value (none) -> RELAY; footprint (none) -> Connector_PinHeader_2.54mm:PinHeader_1x03_P2.54mm_Vertical
- J14: value (none) -> SWITCH; footprint (none) -> TerminalBlock_Phoenix:TerminalBlock_Phoenix_MKDS-1,5-2-5.08_1x02_P5.08mm_Horizontal
- J2: value (none) -> Barrel_Jack_Switch; footprint (none) -> Connector_BarrelJack:BarrelJack_Horizontal
- J3: value (none) -> P+; footprint (none) -> Connector_PinHeader_2.54mm:PinHeader_1x01_P2.54mm_Vertical
- J4: value (none) -> P-; footprint (none) -> Connector_PinHeader_2.54mm:PinHeader_1x01_P2.54mm_Vertical
- J5: value (none) -> B+; footprint (none) -> Connector_PinHeader_2.54mm:PinHeader_1x01_P2.54mm_Vertical
- J6: value (none) -> B2; footprint (none) -> Connector_PinHeader_2.54mm:PinHeader_1x01_P2.54mm_Vertical
- J7: value (none) -> B1; footprint (none) -> Connector_PinHeader_2.54mm:PinHeader_1x01_P2.54mm_Vertical
- J8: value (none) -> B-; footprint (none) -> Connector_PinHeader_2.54mm:PinHeader_1x01_P2.54mm_Vertical
- J9: value (none) -> SENSOR; footprint (none) -> TerminalBlock_Phoenix:TerminalBlock_Phoenix_MKDS-1,5-4-5.08_1x04_P5.08mm_Horizontal
- Q1: value (none) -> BC547; footprint (none) -> Package_TO_SOT_THT:TO-92_Inline
- R1: value (none) -> 3.3k; footprint (none) -> Resistor_THT:R_Axial_DIN0207_L6.3mm_D2.5mm_P10.16mm_Horizontal
- R2: value (none) -> 330; footprint (none) -> Resistor_THT:R_Axial_DIN0207_L6.3mm_D2.5mm_P10.16mm_Horizontal
- U1: value (none) -> L7805; footprint (none) -> Package_TO_SOT_THT:TO-220-3_Vertical
- U2: value (none) -> BOB-12009; footprint (none) -> BOB-12009:CONV_BOB-12009
- U3: value (none) -> BP; footprint (none) -> blue-pill-kicad-master:blue_pill
- U4: value (none) -> Y17P21221FP; footprint (none) -> Y17P21221FP:SW_PVA2EEH21.7NV2
