File: go/go.kicad_sch (KiCad schematic)
At the start: 1 part

Commit message: rasp
Parts:
- added C? (x2): C, symbol Device:C
Other:
- moved on the sheet: U?
Changed lines of the file:
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@@
 (kicad_sch (version 20211123) (generator eeschema)
   (paper "A4")
-  (symbol (lib_id "MCU_ST_STM32F0:STM32F031F6Px") (at 151.13 115.57 0) (unit 1)
+  (symbol (lib_id "Device:C") (at 114.3 92.71 0) (unit 1)
     (in_bom yes) (on_board yes) (fields_autoplaced)
-    (property "Reference" "U?" (id 0) (at 153.1494 135.89 0)
+    (property "Reference" "C?" (id 0) (at 118.11 91.4399 0)
       (effects (font (size 1.27 1.27)) (justify left))
     )
-    (property "Value" "STM32F031F6Px" (id 1) (at 153.1494 138.43 0)
+    (property "Value" "C" (id 1) (at 118.11 93.9799 0)
       (effects (font (size 1.27 1.27)) (justify left))
     )
-    (property "Footprint" "Package_SO:TSSOP-20_4.4x6.5mm_P0.65mm" (id 2) (at 140.97 133.35 0)
+    (property "Footprint" "" (id 2) (at 115.2652 96.52 0)
+      (effects (font (size 1.27 1.27)) hide)
+    )
+    (property "Datasheet" "~" (id 3) (at 114.3 92.71 0)
+      (effects (font (size 1.27 1.27)) hide)
+    )
+    (pin "1")
+    (pin "2")
+  )
+  (symbol (lib_id "MCU_ST_STM32F0:STM32F031F6Px") (at 171.45 102.87 0) (unit 1)
+    (in_bom yes) (on_board yes) (fields_autoplaced)
+    (property "Reference" "U?" (id 0) (at 173.4694 123.19 0)
+      (effects (font (size 1.27 1.27)) (justify left))
+    )
+    (property "Value" "STM32F031F6Px" (id 1) (at 173.4694 125.73 0)
+      (effects (font (size 1.27 1.27)) (justify left))
+    )
+    (property "Footprint" "Package_SO:TSSOP-20_4.4x6.5mm_P0.65mm" (id 2) (at 161.29 120.65 0)
       (effects (font (size 1.27 1.27)) (justify right) hide)
     )
-    (property "Datasheet" "http://www.st.com/st-web-ui/static/active/en/resource/technical/document/datasheet/DM00104043.pdf" (id 3) (at 151.13 115.57 0)
+    (property "Datasheet" "http://www.st.com/st-web-ui/static/active/en/resource/technical/document/datasheet/DM00104043.pdf" (id 3) (at 171.45 102.87 0)
       (effects (font (size 1.27 1.27)) hide)
     )
@@
     (pin "9")
   )
+  (symbol (lib_id "Device:C") (at 125.73 92.71 0) (unit 1)
+    (in_bom yes) (on_board yes) (fields_autoplaced)
+    (property "Reference" "C?" (id 0) (at 129.54 91.4399 0)
+      (effects (font (size 1.27 1.27)) (justify left))
+    )
+    (property "Value" "C" (id 1) (at 129.54 93.9799 0)
+      (effects (font (size 1.27 1.27)) (justify left))
+    )
+    (property "Footprint" "" (id 2) (at 126.6952 96.52 0)
+      (effects (font (size 1.27 1.27)) hide)
+    )
+    (property "Datasheet" "~" (id 3) (at 125.73 92.71 0)
+      (effects (font (size 1.27 1.27)) hide)
+    )
+    (pin "1")
+    (pin "2")
+  )
   (sheet_instances
     (path "/" (page "1"))
   )
   (symbol_instances
+    (path "/143e6104-ac3e-4160-b7d2-1a111dd2b2ad"
+      (reference "C?") (unit 1) (value "C") (footprint "")
+    )
+    (path "/bee3a585-926f-41e5-91ce-a3a04195475b"
+      (reference "C?") (unit 1) (value "C") (footprint "")
+    )
     (path "/1e931afc-ee01-4cf5-ac53-e9b85b0c34ca"
       (reference "U?") (unit 1) (value "STM32F031F6Px") (footprint "Package_SO:TSSOP-20_4.4x6.5mm_P0.65mm")
